File: template/template.kicad_pcb (KiCad board)
At the start: 2 copper layers, 40 x 80 mm, 6 parts

Commit message: WIP
Parts:
- removed NT1, NT2, NT3, NT4: NetTie_2, t80:NetTie-2mm-T80
- removed X2: ~, Connector_PinHeader_2.54mm:PinHeader_2x05_P2.54mm_Vertical
- X1: footprint Connector_PinHeader_2.54mm:PinHeader_2x05_P2.54mm_Vertical -> Connector_IDC:IDC-Header_2x05_P2.54mm_Vertical
- moved X1 1.97 mm to (88.3, 94.9)
Connections:
- X1 pad 1: /PWR_LINE_12V -> GND
- X1 pad 10: /PWR_LINE_3V3 -> +5V
- X1 pad 2: /PWR_LINE_12V -> unconnected-(X1-SCL)
- X1 pad 3: /PWR_LINE_GND -> unconnected-(X1-SDA)
- X1 pad 4: /PWR_LINE_GND -> +3V3
- X1 pad 5: /SCL -> (no net)
- X1 pad 6: /SDA -> (no net)
- X1 pad 7: /RST -> unconnected-(X1-RST)
- X1 pad 8: /IRQ -> unconnected-(X1-IRQ)
- X1 pad 9: /PWR_LINE_5V -> GND
Routing:
- net /PWR_LINE_5V: track 38.0 -> 0.00 mm, vias 1 -> 0
- net /PWR_LINE_3V3: track 38.0 -> 0.00 mm
- net /PWR_LINE_12V: track 37.4 -> 0.00 mm
- net /PWR_LINE_GND: track 37.4 -> 0.00 mm, vias 1 -> 0
- net /IRQ: track 35.9 -> 0.00 mm
- net /RST: track 35.8 -> 0.00 mm, vias 1 -> 0
- net /SDA: track 35.8 -> 0.00 mm
- net /SCL: track 35.8 -> 0.00 mm, vias 1 -> 0
- net GND: track 21.0 -> 0.00 mm, vias 6 -> 0
Other:
- outline, holes or cut-outs redrawn

Commit message: WIP
Parts:
- X1: footprint Connector_IDC:IDC-Header_2x05_P2.54mm_Vertical -> Connector_IDC:IDC-Header_2x04_P2.54mm_Vertical
- moved X1 1.27 mm to (88.3, 96.2)
Connections:
- X1 pad 5: (no net) -> unconnected-(X1-RST)
- X1 pad 6: (no net) -> unconnected-(X1-IRQ)
- X1 pad 7: unconnected-(X1-RST) -> GND
- X1 pad 8: unconnected-(X1-IRQ) -> +5V
Changed lines of the file:
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@@
   (net 6 "unconnected-(X1-IRQ)")
   (net 7 "+5V")
-  (footprint "Connector_IDC:IDC-Header_2x05_P2.54mm_Vertical" (layer "F.Cu")
-    (at 88.29 94.92)
-    (descr "Through hole IDC box header, 2x05, 2.54mm pitch, DIN 41651 / IEC 60603-13, double rows, https://docs.google.com/spreadsheets/d/16SsEcesNF15N3Lb4niX7dcUr-NY5_MFPQhobNuNppn4/edit#gid=0")
-    (tags "Through hole vertical IDC box header THT 2x05 2.54mm double row")
+  (footprint "Connector_IDC:IDC-Header_2x04_P2.54mm_Vertical" (layer "F.Cu")
+    (at 88.29 96.19)
+    (descr "Through hole IDC box header, 2x04, 2.54mm pitch, DIN 41651 / IEC 60603-13, double rows, https://docs.google.com/spreadsheets/d/16SsEcesNF15N3Lb4niX7dcUr-NY5_MFPQhobNuNppn4/edit#gid=0")
+    (tags "Through hole vertical IDC box header THT 2x04 2.54mm double row")
     (property "Sheetfile" "File: template.kicad_sch")
     (property "Sheetname" "")
     (attr through_hole)
-    (fp_text reference "X1" (at 1.27 -6.1) (layer "F.SilkS") hide
+    (fp_text reference "X1" (at 1.27 -6.1) (layer "F.SilkS")
         (effects (font (size 1 1) (thickness 0.15)))
     )
-    (fp_text value "~" (at 1.27 16.26) (layer "F.Fab")
+    (fp_text value "~" (at 1.27 13.72) (layer "F.Fab")
         (effects (font (size 1 1) (thickness 0.15)))
     )
-    (fp_text user "${REFERENCE}" (at 1.27 5.08 90) (layer "F.Fab")
+    (fp_text user "${REFERENCE}" (at 1.27 3.81 90) (layer "F.Fab")
         (effects (font (size 1 1) (thickness 0.15)))
     )
@@
     (fp_line (start -3.29 -5.21) (end 5.83 -5.21)
       (stroke (width 0.12) (type solid)) (layer "F.SilkS"))
-    (fp_line (start -3.29 3.03) (end -1.98 3.03)
+    (fp_line (start -3.29 1.76) (end -1.98 1.76)
       (stroke (width 0.12) (type solid)) (layer "F.SilkS"))
-    (fp_line (start -3.29 15.37) (end -3.29 -5.21)
+    (fp_line (start -3.29 12.83) (end -3.29 -5.21)
       (stroke (width 0.12) (type solid)) (layer "F.SilkS"))
     (fp_line (start -1.98 -3.91) (end 4.52 -3.91)
       (stroke (width 0.12) (type solid)) (layer "F.SilkS"))
-    (fp_line (start -1.98 3.03) (end -1.98 -3.91)
+    (fp_line (start -1.98 1.76) (end -1.98 -3.91)
       (stroke (width 0.12) (type solid)) (layer "F.SilkS"))
-    (fp_line (start -1.98 7.13) (end -3.29 7.13)
+    (fp_line (start -1.98 5.86) (end -3.29 5.86)
       (stroke (width 0.12) (type solid)) (layer "F.SilkS"))
-    (fp_line (start -1.98 7.13) (end -1.98 7.13)
+    (fp_line (start -1.98 5.86) (end -1.98 5.86)
       (stroke (width 0.12) (type solid)) (layer "F.SilkS"))
-    (fp_line (start -1.98 14.07) (end -1.98 7.13)
+    (fp_line (start -1.98 11.53) (end -1.98 5.86)
       (stroke (width 0.12) (type solid)) (layer "F.SilkS"))
-    (fp_line (start 4.52 -3.91) (end 4.52 14.07)
+    (fp_line (start 4.52 -3.91) (end 4.52 11.53)
       (stroke (width 0.12) (type solid)) (layer "F.SilkS"))
-    (fp_line (start 4.52 14.07) (end -1.98 14.07)
+    (fp_line (start 4.52 11.53) (end -1.98 11.53)
       (stroke (width 0.12) (type solid)) (layer "F.SilkS"))
-    (fp_line (start 5.83 -5.21) (end 5.83 15.37)
+    (fp_line (start 5.83 -5.21) (end 5.83 12.83)
       (stroke (width 0.12) (type solid)) (layer "F.SilkS"))
-    (fp_line (start 5.83 15.37) (end -3.29 15.37)
+    (fp_line (start 5.83 12.83) (end -3.29 12.83)
       (stroke (width 0.12) (type solid)) (layer "F.SilkS"))
-    (fp_line (start -3.68 -5.6) (end -3.68 15.76)
+    (fp_line (start -3.68 -5.6) (end -3.68 13.22)
       (stroke (width 0.05) (type solid)) (layer "F.CrtYd"))
-    (fp_line (start -3.68 15.76) (end 6.22 15.76)
+    (fp_line (start -3.68 13.22) (end 6.22 13.22)
       (stroke (width 0.05) (type solid)) (layer "F.CrtYd"))
     (fp_line (start 6.22 -5.6) (end -3.68 -5.6)
       (stroke (width 0.05) (type solid)) (layer "F.CrtYd"))
-    (fp_line (start 6.22 15.76) (end 6.22 -5.6)
+    (fp_line (start 6.22 13.22) (end 6.22 -5.6)
       (stroke (width 0.05) (type solid)) (layer "F.CrtYd"))
     (fp_line (start -3.18 -4.1) (end -2.18 -5.1)
       (stroke (width 0.1) (type solid)) (layer "F.Fab"))
-    (fp_line (start -3.18 3.03) (end -1.98 3.03)
+    (fp_line (start -3.18 1.76) (end -1.98 1.76)
       (stroke (width 0.1) (type solid)) (layer "F.Fab"))
-    (fp_line (start -3.18 15.26) (end -3.18 -4.1)
+    (fp_line (start -3.18 12.72) (end -3.18 -4.1)
       (stroke (width 0.1) (type solid)) (layer "F.Fab"))
     (fp_line (start -2.18 -5.1) (end 5.72 -5.1)
@@
     (fp_line (start -1.98 -3.91) (end 4.52 -3.91)
       (stroke (width 0.1) (type solid)) (layer "F.Fab"))
-    (fp_line (start -1.98 3.03) (end -1.98 -3.91)
+    (fp_line (start -1.98 1.76) (end -1.98 -3.91)
       (stroke (width 0.1) (type solid)) (layer "F.Fab"))
-    (fp_line (start -1.98 7.13) (end -3.18 7.13)
+    (fp_line (start -1.98 5.86) (end -3.18 5.86)
       (stroke (width 0.1) (type solid)) (layer "F.Fab"))
-    (fp_line (start -1.98 7.13) (end -1.98 7.13)
+    (fp_line (start -1.98 5.86) (end -1.98 5.86)
       (stroke (width 0.1) (type solid)) (layer "F.Fab"))
-    (fp_line (start -1.98 14.07) (end -1.98 7.13)
+    (fp_line (start -1.98 11.53) (end -1.98 5.86)
       (stroke (width 0.1) (type solid)) (layer "F.Fab"))
-    (fp_line (start 4.52 -3.91) (end 4.52 14.07)
+    (fp_line (start 4.52 -3.91) (end 4.52 11.53)
       (stroke (width 0.1) (type solid)) (layer "F.Fab"))
-    (fp_line (start 4.52 14.07) (end -1.98 14.07)
+    (fp_line (start 4.52 11.53) (end -1.98 11.53)
       (stroke (width 0.1) (type solid)) (layer "F.Fab"))
-    (fp_line (start 5.72 -5.1) (end 5.72 15.26)
+    (fp_line (start 5.72 -5.1) (end 5.72 12.72)
       (stroke (width 0.1) (type solid)) (layer "F.Fab"))
-    (fp_line (start 5.72 15.26) (end -3.18 15.26)
+    (fp_line (start 5.72 12.72) (end -3.18 12.72)
       (stroke (width 0.1) (type solid)) (layer "F.Fab"))
     (pad "1" thru_hole roundrect (at 0 0) (size 1.7 1.7) (drill 1) (layers *.Cu *.Mask) (roundrect_rratio 0.147059)
@@
     (pad "4" thru_hole circle (at 2.54 2.54) (size 1.7 1.7) (drill 1) (layers *.Cu *.Mask)
       (net 3 "+3V3") (pinfunction "3V3") (pintype "power_out"))
-    (pad "5" thru_hole circle (at 0 5.08) (size 1.7 1.7) (drill 1) (layers *.Cu *.Mask))
-    (pad "6" thru_hole circle (at 2.54 5.08) (size 1.7 1.7) (drill 1) (layers *.Cu *.Mask))
+    (pad "5" thru_hole circle (at 0 5.08) (size 1.7 1.7) (drill 1) (layers *.Cu *.Mask)
+      (net 5 "unconnected-(X1-RST)") (pinfunction "RST") (pintype "bidirectional+no_connect"))
+    (pad "6" thru_hole circle (at 2.54 5.08) (size 1.7 1.7) (drill 1) (layers *.Cu *.Mask)
+      (net 6 "unconnected-(X1-IRQ)") (pinfunction "IRQ") (pintype "bidirectional+no_connect"))
     (pad "7" thru_hole circle (at 0 7.62) (size 1.7 1.7) (drill 1) (layers *.Cu *.Mask)
-      (net 5 "unconnected-(X1-RST)") (pinfunction "RST") (pintype "bidirectional+no_connect"))
+      (net 4 "GND") (pinfunction "GND") (pintype "power_out"))
     (pad "8" thru_hole circle (at 2.54 7.62) (size 1.7 1.7) (drill 1) (layers *.Cu *.Mask)
-      (net 6 "unconnected-(X1-IRQ)") (pinfunction "IRQ") (pintype "bidirectional+no_connect"))
-    (pad "9" thru_hole circle (at 0 10.16) (size 1.7 1.7) (drill 1) (layers *.Cu *.Mask)
-      (net 4 "GND") (pinfunction "GND") (pintype "power_out"))
-    (pad "10" thru_hole circle (at 2.54 10.16) (size 1.7 1.7) (drill 1) (layers *.Cu *.Mask)
       (net 7 "+5V") (pinfunction "5V") (pintype "power_out"))
-    (model "${KICAD6_3DMODEL_DIR}/Connector_IDC.3dshapes/IDC-Header_2x05_P2.54mm_Vertical.wrl"
+    (model "${KICAD6_3DMODEL_DIR}/Connector_IDC.3dshapes/IDC-Header_2x04_P2.54mm_Vertical.wrl"
       (offset (xyz 0 0 0))
       (scale (xyz 1 1 1))
