File: template/template.kicad_sch (KiCad schematic)
At the start: 7 parts

Commit message: WIP
Parts:
- removed NT1: NetTie_2, symbol Device:NetTie_2
Changed lines of the file:
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@@
-(kicad_sch (version 20220904) (generator eeschema)
+(kicad_sch (version 20220914) (generator eeschema)
   (paper "A4")
-  (junction (at 154.94 185.42) (diameter 0) (color 0 0 0 0)
-  )
-  (junction (at 160.02 185.42) (diameter 0) (color 0 0 0 0)
-  )
-  (wire (pts (xy 154.94 185.42) (xy 154.94 187.96))
-    (stroke (width 0) (type default))
-  )
   (wire (pts (xy 139.7 177.8) (xy 154.94 177.8))
     (stroke (width 0) (type default))
@@
     (stroke (width 0) (type default))
   )
-  (wire (pts (xy 160.02 185.42) (xy 160.02 187.96))
-    (stroke (width 0) (type default))
-  )
   (wire (pts (xy 139.7 185.42) (xy 154.94 185.42))
     (stroke (width 0) (type default))
@@
   )
   (symbol (lib_id "t80:t80-pin-header") (at 93.98 170.18 0) (unit 1)
-    (in_bom yes) (on_board yes) (fields_autoplaced)
+    (in_bom yes) (on_board yes) (dnp no) (fields_autoplaced)
     (default_instance (reference "X1") (unit 1) (value "~") (footprint ""))
     (property "Reference" "X1" (id 0) (at 93.98 161.9123 0)
@@
   )
   (symbol (lib_id "power:PWR_FLAG") (at 160.02 162.56 90) (unit 1)
-    (in_bom yes) (on_board yes) (fields_autoplaced)
+    (in_bom yes) (on_board yes) (dnp no) (fields_autoplaced)
     (default_instance (reference "#FLG?") (unit 1) (value "PWR_FLAG") (footprint ""))
     (property "Reference" "#FLG?" (id 0) (at 158.115 162.56 0)
@@
   )
   (symbol (lib_id "Device:NetTie_2") (at 157.48 177.8 0) (unit 1)
-    (in_bom yes) (on_board yes) (fields_autoplaced)
+    (in_bom yes) (on_board yes) (dnp no) (fields_autoplaced)
     (default_instance (reference "NT1") (unit 1) (value "NetTie_2") (footprint ""))
     (property "Reference" "NT1" (id 0) (at 157.48 176.7301 0)
@@
   )
   (symbol (lib_id "power:PWR_FLAG") (at 160.02 167.64 90) (unit 1)
-    (in_bom yes) (on_board yes) (fields_autoplaced)
+    (in_bom yes) (on_board yes) (dnp no) (fields_autoplaced)
     (default_instance (reference "#FLG?") (unit 1) (value "PWR_FLAG") (footprint ""))
     (property "Reference" "#FLG?" (id 0) (at 158.115 167.64 0)
@@
   )
   (symbol (lib_id "power:PWR_FLAG") (at 139.7 182.88 90) (unit 1)
-    (in_bom yes) (on_board yes) (fields_autoplaced)
+    (in_bom yes) (on_board yes) (dnp no) (fields_autoplaced)
     (default_instance (reference "#FLG?") (unit 1) (value "PWR_FLAG") (footprint ""))
     (property "Reference" "#FLG?" (id 0) (at 137.795 182.88 0)
@@
   )
   (symbol (lib_id "power:GND") (at 160.02 170.18 90) (unit 1)
-    (in_bom yes) (on_board yes) (fields_autoplaced)
+    (in_bom yes) (on_board yes) (dnp no) (fields_autoplaced)
     (default_instance (reference "#PWR?") (unit 1) (value "GND") (footprint ""))
     (property "Reference" "#PWR?" (id 0) (at 166.37 170.18 0)
@@
   )
   (symbol (lib_id "power:+12V") (at 160.02 177.8 270) (unit 1)
-    (in_bom yes) (on_board yes) (fields_autoplaced)
+    (in_bom yes) (on_board yes) (dnp no) (fields_autoplaced)
     (default_instance (reference "#PWR?") (unit 1) (value "+12V") (footprint ""))
     (property "Reference" "#PWR?" (id 0) (at 156.21 177.8 0)
@@
   )
   (symbol (lib_id "Device:NetTie_2") (at 157.48 182.88 0) (unit 1)
-    (in_bom yes) (on_board yes) (fields_autoplaced)
+    (in_bom yes) (on_board yes) (dnp no) (fields_autoplaced)
     (default_instance (reference "NT1") (unit 1) (value "NetTie_2") (footprint ""))
     (property "Reference" "NT1" (id 0) (at 157.48 181.8101 0)
@@
   )
   (symbol (lib_id "power:GND") (at 160.02 185.42 90) (unit 1)
-    (in_bom yes) (on_board yes) (fields_autoplaced)
+    (in_bom yes) (on_board yes) (dnp no) (fields_autoplaced)
     (default_instance (reference "#PWR?") (unit 1) (value "GND") (footprint ""))
     (property "Reference" "#PWR?" (id 0) (at 166.37 185.42 0)
@@
   )
   (symbol (lib_id "power:+5V") (at 160.02 180.34 270) (unit 1)
-    (in_bom yes) (on_board yes) (fields_autoplaced)
+    (in_bom yes) (on_board yes) (dnp no) (fields_autoplaced)
     (default_instance (reference "#PWR?") (unit 1) (value "+5V") (footprint ""))
     (property "Reference" "#PWR?" (id 0) (at 156.21 180.34 0)
@@
   )
   (symbol (lib_id "power:+5V") (at 160.02 165.1 270) (unit 1)
-    (in_bom yes) (on_board yes) (fields_autoplaced)
+    (in_bom yes) (on_board yes) (dnp no) (fields_autoplaced)
     (default_instance (reference "#PWR?") (unit 1) (value "+5V") (footprint ""))
     (property "Reference" "#PWR?" (id 0) (at 156.21 165.1 0)
@@
   )
   (symbol (lib_id "power:PWR_FLAG") (at 139.7 185.42 90) (unit 1)
-    (in_bom yes) (on_board yes) (fields_autoplaced)
+    (in_bom yes) (on_board yes) (dnp no) (fields_autoplaced)
     (default_instance (reference "#FLG?") (unit 1) (value "PWR_FLAG") (footprint ""))
     (property "Reference" "#FLG?" (id 0) (at 137.795 185.42 0)
@@
   )
   (symbol (lib_id "power:PWR_FLAG") (at 139.7 180.34 90) (unit 1)
-    (in_bom yes) (on_board yes) (fields_autoplaced)
+    (in_bom yes) (on_board yes) (dnp no) (fields_autoplaced)
     (default_instance (reference "#FLG?") (unit 1) (value "PWR_FLAG") (footprint ""))
     (property "Reference" "#FLG?" (id 0) (at 137.795 180.34 0)
@@
   )
   (symbol (lib_id "t80:t80-pin-header") (at 43.18 170.18 0) (unit 1)
-    (in_bom yes) (on_board yes) (fields_autoplaced)
+    (in_bom yes) (on_board yes) (dnp no) (fields_autoplaced)
     (default_instance (reference "X1") (unit 1) (value "~") (footprint ""))
     (property "Reference" "X1" (id 0) (at 43.18 161.9123 0)
@@
   )
   (symbol (lib_id "Device:NetTie_2") (at 157.48 185.42 0) (unit 1)
-    (in_bom yes) (on_board yes) (fields_autoplaced)
+    (in_bom yes) (on_board yes) (dnp no) (fields_autoplaced)
     (default_instance (reference "NT1") (unit 1) (value "NetTie_2") (footprint ""))
     (property "Reference" "NT1" (id 0) (at 157.48 184.3501 0)
@@
   )
   (symbol (lib_id "power:PWR_FLAG") (at 139.7 177.8 90) (unit 1)
-    (in_bom yes) (on_board yes) (fields_autoplaced)
+    (in_bom yes) (on_board yes) (dnp no) (fields_autoplaced)
     (default_instance (reference "#FLG?") (unit 1) (value "PWR_FLAG") (footprint ""))
     (property "Reference" "#FLG?" (id 0) (at 137.795 177.8 0)
@@
   )
   (symbol (lib_id "power:+3V3") (at 160.02 167.64 270) (unit 1)
-    (in_bom yes) (on_board yes) (fields_autoplaced)
+    (in_bom yes) (on_board yes) (dnp no) (fields_autoplaced)
     (default_instance (reference "#PWR?") (unit 1) (value "+3V3") (footprint ""))
     (property "Reference" "#PWR?" (id 0) (at 156.21 167.64 0)
@@
     (pin "1")
   )
-  (symbol (lib_id "Device:NetTie_2") (at 157.48 187.96 0) (unit 1)
-    (in_bom yes) (on_board yes) (fields_autoplaced)
-    (default_instance (reference "NT1") (unit 1) (value "NetTie_2") (footprint ""))
-    (property "Reference" "NT1" (id 0) (at 157.48 186.8901 0)
-      (effects (font (size 1.27 1.27)))
-    )
-    (property "Value" "NetTie_2" (id 1) (at 157.48 186.8901 0)
-      (effects (font (size 1.27 1.27)) hide)
-    )
-    (property "Footprint" "" (id 2) (at 157.48 187.96 0)
-      (effects (font (size 1.27 1.27)) hide)
-    )
-    (property "Datasheet" "~" (id 3) (at 157.48 187.96 0)
-      (effects (font (size 1.27 1.27)) hide)
-    )
-    (pin "1")
-    (pin "2")
-  )
   (symbol (lib_id "power:+12V") (at 160.02 162.56 270) (unit 1)
-    (in_bom yes) (on_board yes) (fields_autoplaced)
+    (in_bom yes) (on_board yes) (dnp no) (fields_autoplaced)
     (default_instance (reference "#PWR?") (unit 1) (value "+12V") (footprint ""))
     (property "Reference" "#PWR?" (id 0) (at 156.21 162.56 0)
@@
   )
   (symbol (lib_id "power:+3V3") (at 160.02 182.88 270) (unit 1)
-    (in_bom yes) (on_board yes) (fields_autoplaced)
+    (in_bom yes) (on_board yes) (dnp no) (fields_autoplaced)
     (default_instance (reference "#PWR?") (unit 1) (value "+3V3") (footprint ""))
     (property "Reference" "#PWR?" (id 0) (at 156.21 182.88 0)
@@
   )
   (symbol (lib_id "power:PWR_FLAG") (at 160.02 165.1 90) (unit 1)
-    (in_bom yes) (on_board yes) (fields_autoplaced)
+    (in_bom yes) (on_board yes) (dnp no) (fields_autoplaced)
     (default_instance (reference "#FLG?") (unit 1) (value "PWR_FLAG") (footprint ""))
     (property "Reference" "#FLG?" (id 0) (at 158.115 165.1 0)
@@
   )
   (symbol (lib_id "power:PWR_FLAG") (at 160.02 170.18 90) (unit 1)
-    (in_bom yes) (on_board yes) (fields_autoplaced)
+    (in_bom yes) (on_board yes) (dnp no) (fields_autoplaced)
     (default_instance (reference "#FLG?") (unit 1) (value "PWR_FLAG") (footprint ""))
     (property "Reference" "#FLG?" (id 0) (at 158.115 170.18 0)
@@
   )
   (symbol (lib_id "Device:NetTie_2") (at 157.48 180.34 0) (unit 1)
-    (in_bom yes) (on_board yes) (fields_autoplaced)
+    (in_bom yes) (on_board yes) (dnp no) (fields_autoplaced)
     (default_instance (reference "NT1") (unit 1) (value "NetTie_2") (footprint ""))
     (property "Reference" "NT1" (id 0) (at 157.48 179.2701 0)
@@
     )
     (path "/28916dd8-f213-404d-a954-2fe9c318e4cb"
-      (reference "NT1") (unit 1) (value "NetTie_2") (footprint "t80:NetTie-2_SMD_Pad2mm-T80")
+      (reference "NT1") (unit 1) (value "NetTie_2") (footprint "t80:NetTie-2mm-T80")
     )
     (path "/fbc33482-bb11-4339-9850-a56d848eee4c"
-      (reference "NT2") (unit 1) (value "NetTie_2") (footprint "t80:NetTie-2_SMD_Pad0.25mm-T80")
+      (reference "NT2") (unit 1) (value "NetTie_2") (footprint "t80:NetTie-2mm-T80")
     )
     (path "/5b633814-ddc2-4d6f-aff0-4efc9aa9a231"
-      (reference "NT3") (unit 1) (value "NetTie_2") (footprint "t80:NetTie-2_SMD_Pad0.25mm-T80")
+      (reference "NT3") (unit 1) (value "NetTie_2") (footprint "t80:NetTie-2mm-T80")
     )
     (path "/a1bd9c37-3874-4bc4-a32c-bd7e2b30e4b1"
-      (reference "NT4") (unit 1) (value "NetTie_2") (footprint "t80:NetTie-2_SMD_Pad2mm-T80")
-    )
-    (path "/da1f327b-cf13-4365-a02d-f2a050029507"
-      (reference "NT5") (unit 1) (value "NetTie_2") (footprint "t80:NetTie-2_SMD_Pad2mm-T80")
+      (reference "NT4") (unit 1) (value "NetTie_2") (footprint "t80:NetTie-2mm-T80")
     )
     (path "/9cd4ee06-f76a-4022-9705-d1ca8fd213d3"

Commit message: WIP
Parts:
- removed NT1 (x4): NetTie_2, symbol Device:NetTie_2
- removed X1: ~, symbol t80:t80-pin-header
Connections:
- net PWR_LINE_3V3 is gone; now on net +5V: X1.10 (5V)
- net PWR_LINE_5V is gone; now on net GND: X1.9 (GND)
- net +3V3: now also X1.4 (3V3)
- net GND: now also X1.1 (GND)
- net IRQ: no longer names the net of X1.8 (IRQ)
- net PWR_LINE_12V: no longer names the net of X1.2 (SCL)
- net PWR_LINE_12V: no longer X1.1 (12V)
- net PWR_LINE_GND: no longer names the net of X1.3 (SDA)
- net PWR_LINE_GND: no longer X1.4 (GND)
- net RST: no longer names the net of X1.7 (RST)
- removed net SCL: X1.5 (SCL)
- removed net SDA: X1.6 (SDA)
- no-connect marks 0 -> 4

Commit message: WIP
Connections:
- net +5V: now also X1.8 (5V); no longer X1.10 (5V)
- net GND: now also X1.7 (GND); no longer X1.9 (GND)
Changed lines of the file:
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@@
   (no_connect (at 50.8 175.26))
   (no_connect (at 50.8 172.72))
+  (no_connect (at 50.8 167.64))
   (no_connect (at 50.8 170.18))
-  (no_connect (at 50.8 167.64))
   (wire (pts (xy 40.64 185.42) (xy 43.18 185.42))
     (stroke (width 0) (type default))
@@
     )
     (pin "1")
-    (pin "10")
     (pin "2")
     (pin "3")
     (pin "4")
+    (pin "5")
+    (pin "6")
     (pin "7")
     (pin "8")
-    (pin "9")
   )
   (symbol (lib_id "power:+3V3") (at 40.64 157.48 0) (unit 1)
@@
     )
     (path "/9cd4ee06-f76a-4022-9705-d1ca8fd213d3"
-      (reference "X1") (unit 1) (value "~") (footprint "Connector_IDC:IDC-Header_2x05_P2.54mm_Vertical")
+      (reference "X1") (unit 1) (value "~") (footprint "Connector_IDC:IDC-Header_2x04_P2.54mm_Vertical")
     )
   )
